File: expansion-backplane/hardware/expansion-connector/expansion-connector.kicad_sch (KiCad schematic)
At the start: 2 parts

Commit message: updatedd PCB layouts
Parts:
- CN1, CN2: footprint Connector_PinSocket_2.54mm:PinSocket_2x32_P2.54mm_Vertical -> Connector_PinHeader_2.54mm:PinHeader_2x16_P2.54mm_Vertical
Changed lines of the file:
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@@
 			)
 		)
-		(property "Footprint" "Connector_PinSocket_2.54mm:PinSocket_2x32_P2.54mm_Vertical"
+		(property "Footprint" "Connector_PinHeader_2.54mm:PinHeader_2x16_P2.54mm_Vertical"
 			(at 222.504 13.97 0)
 			(effects
@@
 			)
 		)
-		(property "Footprint" "Connector_PinSocket_2.54mm:PinSocket_2x32_P2.54mm_Vertical"
+		(property "Footprint" "Connector_PinHeader_2.54mm:PinHeader_2x16_P2.54mm_Vertical"
 			(at 167.894 13.97 0)
 			(effects
