File: multiplier/hardware/four-bit-multiplier/four-bit-multiplier.kicad_sch (KiCad schematic)
At the start: 20 parts, among them J1 Conn_01x08_Pin, SW2 SW_DIP_x04, SW3 SW_DIP_x04, U1 74LS32, U2 74LS32, U3 74LS283, U4 74LS32, U5 74LS283, U6 74LS32, U7 74LS283

Commit message: fixed carry
Connections:
- net GND: now also U3.12 (A4)
Other:
- moved on the sheet: C1, C2, C3, C4, C5, C6, C7, C8, J1, RN2, RN3, SW2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

Commit message: first version of multiplier board
Parts:
- removed C8: 0.1 µF, symbol Device:C
- removed J1: Conn_01x08_Pin, symbol Connector:Conn_01x08_Pin
- removed RN2, RN3: R_Network04, Resistor_THT:R_Array_SIP5, symbol Device:R_Network04
- removed SW2, SW3: SW_DIP_x04, symbol Switch:SW_DIP_x04
- removed U1, U2, U4, U6: 74LS32, symbol 74xx:74LS32
- added J1, J2: Conn_01x09_Pin, Connector_PinHeader_2.54mm:PinHeader_1x09_P2.54mm_Vertical, symbol Connector:Conn_01x09_Pin
- added U1, U2, U4, U6: 74AHCT08, Package_SO:SOIC-14_3.9x8.7mm_P1.27mm, symbol 74xx:74LS08
- C1, C2, C3, C4, C5, C6, C7: footprint (none) -> Capacitor_SMD:C_0805_2012Metric_Pad1.18x1.45mm_HandSolder
- U3, U5, U7: value 74LS283 -> 74HCT283; footprint (none) -> Package_SO:SOIC-16_3.9x9.9mm_P1.27mm
Connections:
- net +5V: now also J1.1 (Pin_1), U1.14 (VCC), U2.14 (VCC), U4.14 (VCC), U6.14 (VCC)
- net GND: now also J2.1 (Pin_1), U1.7 (GND), U2.7 (GND), U4.7 (GND), U6.7 (GND)
- net at U7.11 (B4): now also U6.11
- net at U5.6 (B1): now also U4.3
- net at U3.11 (B4): now also U1.11
- net at U3.14 (A3): now also U2.11
- net at U3.15 (B3): now also U1.8
- net at U3.2 (B2): now also U1.6
- net at U3.3 (A2): now also U2.8
- net R1: now reaches U3.4 (S1)
- net R1: now also J2.8 (Pin_8)
- net at U3.5 (A1): now also U2.6
- net at U3.6 (B1): now also U1.3
- net at U5.15 (B3): now also U4.8
- net at U7.2 (B2): now also U6.6
- net R4: now reaches U7.1 (S2)
- net R4: now also J2.5 (Pin_5)
- net R6: now reaches U7.10 (S4)
- net R6: now also J2.3 (Pin_3)
- net R5: now reaches U7.13 (S3)
- net R5: now also J2.4 (Pin_4)
- net at U7.15 (B3): now also U6.8
- net R3: now reaches U7.4 (S1)
- net R3: now also J2.6 (Pin_6)
- net at U7.6 (B1): now also U6.3
- net R7: now reaches U7.9 (C4)
- net R7: now also J2.2 (Pin_2)
- net at U5.2 (B2): now also U4.6
- net at U5.11 (B4): now also U4.11
- net R2: now reaches U5.4 (S1)
- net R2: now also J2.7 (Pin_7)
- new net A0: J1.5 (Pin_5), U1.2, U2.2, U4.2, U6.2
- new net A1: J1.4 (Pin_4), U1.5, U2.5, U4.5, U6.5
- new net A2: J1.3 (Pin_3), U1.10, U2.10, U4.10, U6.10
- new net A3: J1.2 (Pin_2), U1.13, U2.13, U4.13, U6.13
- new net B0: J1.9 (Pin_9), U2.1, U2.12, U2.4, U2.9
- new net B1: J1.8 (Pin_8), U1.1, U1.12, U1.4, U1.9
- new net B2: J1.7 (Pin_7), U4.1, U4.12, U4.4, U4.9
- new net B3: J1.6 (Pin_6), U6.1, U6.12, U6.4, U6.9
- new net R0: J2.9 (Pin_9), U2.3
Other:
- note removed: "A Value"
- note removed: "B Value"
