File: multiplier/hardware/multiplier-board/multiplier-board.kicad_sch (KiCad schematic)
At the start: 80 parts, among them U1 74AHCT08, U10 74HCT688, U11 74AHCT08, U12 74AHCT08, U13 74AHCT08, U14 74AHCT08, U15 74AHCT08, U16 74AHCT08, U17 74AHCT08, U18 74AHCT08, U19 ATF16V10C, U2 74AHCT08, U20 74AHCT374, U21 74LS283, U22 74LS283, U23 74LS283, U24 74LS283, U25 74LS283, U26 74LS283, U27 74LS283, U28 74AHCT374, U29 74LS283, U3 74AHCT08, U30 74LS283, U31 74LS283, U32 74LS283, U33 74LS283, U34 74LS283, U35 74LS283, U36 74AHCT245, U37 74AHCT245, U4 74AHCT08, U5 74AHCT08, U6 74AHCT08, U7 74AHCT08, U8 74AHCT08, U9 74HCT688

Commit message: corrected part designator
Parts:
- U21, U22, U23, U24, U25, U26, U27, U29, U30, U31, U32, U33, U34, U35: value 74LS283 -> 74HCT283
Changed lines of the file:
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@@
 			)
 		)
-		(property "Value" "74LS283"
+		(property "Value" "74HCT283"
 			(at 266.7 414.9203 90)
 			(effects
@@
 			)
 		)
-		(property "Value" "74LS283"
+		(property "Value" "74HCT283"
 			(at 266.7 179.9703 90)
 			(effects
@@
 			)
 		)
-		(property "Value" "74LS283"
+		(property "Value" "74HCT283"
 			(at 266.7 132.9803 90)
 			(effects
@@
 			)
 		)
-		(property "Value" "74LS283"
+		(property "Value" "74HCT283"
 			(at 215.9 414.9203 90)
 			(effects
@@
 			)
 		)
-		(property "Value" "74LS283"
+		(property "Value" "74HCT283"
 			(at 215.9 132.9803 90)
 			(effects
@@
 			)
 		)
-		(property "Value" "74LS283"
+		(property "Value" "74HCT283"
 			(at 215.9 273.9503 90)
 			(effects
@@
 			)
 		)
-		(property "Value" "74LS283"
+		(property "Value" "74HCT283"
 			(at 266.7 320.9403 90)
 			(effects
@@
 			)
 		)
-		(property "Value" "74LS283"
+		(property "Value" "74HCT283"
 			(at 215.9 367.9303 90)
 			(effects
@@
 			)
 		)
-		(property "Value" "74LS283"
+		(property "Value" "74HCT283"
 			(at 266.7 226.9603 90)
 			(effects
@@
 			)
 		)
-		(property "Value" "74LS283"
+		(property "Value" "74HCT283"
 			(at 266.7 273.9503 90)
 			(effects
@@
 			)
 		)
-		(property "Value" "74LS283"
+		(property "Value" "74HCT283"
 			(at 215.9 226.9603 90)
 			(effects
@@
 			)
 		)
-		(property "Value" "74LS283"
+		(property "Value" "74HCT283"
 			(at 215.9 179.9703 90)
 			(effects
@@
 			)
 		)
-		(property "Value" "74LS283"
+		(property "Value" "74HCT283"
 			(at 215.9 320.9403 90)
 			(effects
@@
 			)
 		)
-		(property "Value" "74LS283"
+		(property "Value" "74HCT283"
 			(at 266.7 367.9303 90)
 			(effects

Commit message: added controller PLD
Parts:
- U19: value ATF16V10C -> ATF16V8C
Connections:
- net RHIGH: now reaches U19.14 (I/O), U36.19 (CE)
- net BIN: now reaches U19.13 (I/O), U28.11 (Cp)
- net AIN: now reaches U19.12 (I/O), U20.11 (Cp)
- net RLOW: now reaches U19.15 (I/O), U37.19 (CE)
- net ADDR_HIGH: now reaches U19.6 (I5), U9.19 (P=R)
Changed lines of the file:
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@@
 		)
 	)
+	(label "BIN"
+		(at 149.86 473.71 0)
+		(effects
+			(font
+				(size 1.27 1.27)
+			)
+			(justify left bottom)
+		)
+	)
 	(label "BUS0"
 		(at 199.39 515.62 90)
@@
 		)
 	)
+	(label "ADDR_HIGH"
+		(at 38.1 421.64 0)
+		(effects
+			(font
+				(size 1.27 1.27)
+			)
+			(justify left bottom)
+		)
+	)
 	(label "BUS4"
 		(at 132.08 553.72 90)
@@
 		)
 	)
+	(label "RHIGH"
+		(at 149.86 471.17 0)
+		(effects
+			(font
+				(size 1.27 1.27)
+			)
+			(justify left bottom)
+		)
+	)
 	(label "BUS3"
 		(at 191.77 515.62 90)
@@
 		)
 	)
+	(label "AIN"
+		(at 149.86 476.25 0)
+		(effects
+			(font
+				(size 1.27 1.27)
+			)
+			(justify left bottom)
+		)
+	)
 	(label "BUS0"
 		(at 303.53 515.62 90)
@@
 		)
 	)
+	(label "RLOW"
+		(at 149.86 468.63 0)
+		(effects
+			(font
+				(size 1.27 1.27)
+			)
+			(justify left bottom)
+		)
+	)
 	(label "BUS6"
 		(at 340.36 515.62 90)
@@
 			)
 		)
-		(property "Value" "ATF16V10C"
+		(property "Value" "ATF16V8C"
 			(at 136.652 452.3048 0)
 			(effects
