File: timer/hardware/timer/timer.kicad_sch (KiCad schematic)
At the start: 26 parts, among them U1 74HC590, U2 74HC590, U3 74HC590, U4 74HC590, U5 74HC590, U6 74HC590, U7 74HC688, U8 74HC688, U9 ATF22V10C

Commit message: timer pcb layout
Parts:
- removed JP1: Jumper_2_Open, Connector_PinHeader_2.54mm:PinHeader_1x02_P2.54mm_Vertical, symbol Jumper:Jumper_2_Open
- removed JP2, JP3, JP4, JP5: Jumper_2_Bridged, Connector_PinHeader_2.54mm:PinHeader_1x02_P2.54mm_Vertical, symbol Jumper:Jumper_2_Bridged
- added J1: Conn_02x05_Odd_Even, Connector_PinHeader_2.54mm:PinHeader_2x05_P2.54mm_Vertical, symbol Connector_Generic:Conn_02x05_Odd_Even
- C1, C2, C3, C4, C5, C6, C7, C8, C9: footprint (none) -> Capacitor_THT:C_Disc_D3.4mm_W2.1mm_P2.50mm
- renumbered RN2 to RN1, RN1 to RN2
Connections:
- net +5V: now also J1.1 (Pin_1), J1.3 (Pin_3), J1.5 (Pin_5), J1.7 (Pin_7), J1.9 (Pin_9)
- net A0: now also U9.4 (PD/IN3); no longer U9.2 (IN1)
- net A2: now also U9.2 (IN1); no longer U9.4 (PD/IN3)
- net at RN2.6 (R5), U8.3 (R0): now also J1.10 (Pin_10)
- net at RN2.2 (R1), U8.12 (R4): now also J1.2 (Pin_2)
- net at RN2.3 (R2), U8.9 (R3): now also J1.4 (Pin_4)
- net at RN2.4 (R3), U8.7 (R2): now also J1.6 (Pin_6)
- net at RN2.5 (R4), U8.5 (R1): now also J1.8 (Pin_8)
